File: arm.kicad_sch (KiCad schematic)
At the start: 33 parts, among them J1 TC2030-IDC-NL, U10 MX25V1006FZUI, U11 MIC5528-3.3, U4 STM32F042G6Ux, U6 KTD2026EWE-TR, U7 ATA6561-GBQW-N, U8 AP63205WU

Commit message: Update MPNs and add jlcpcb comments.
Parts:
- C11, C14, C15, C16, C19, C20, C27: CAPACITANCE 100 nF -> (none); CAPACITANCE TOLERANCE ±10% -> (none); CASE/PACKAGE 0402 -> (none); CASE/PACKAGE (SI) 1005 -> (none); DIELECTRIC CHARACTERISTIC X7R -> (none); DIELECTRIC MATERIAL Ceramic Multilayer -> (none); FOOTPRINT PCB-ya5qsrmvtd5pjczft90h-1 -> (none); JLCPCB Comment (none) -> 100nF 50V X7R; JLCPCB Footprint (none) -> 0402; LEAD-FREE STATUS Lead Free -> (none); MANUFACTURER PART NUMBER C1005X7R1C104K050BC -> (none); MOUNTING STYLE Surface Mount -> (none); MPN (none) -> GMC04X7R104K50NT; NUMBER OF PINS 2 -> (none); OCTOPART URL http://octopart.com/c1005x7r1c104k050bc-tdk-25947551 -> (none); OCTOPARTID f7023f833ffb28c5 -> (none); PACKAGING Cut Tape (CT), Tape & Reel (TR) -> (none); ROHS Compliant -> (none); SIZE-LENGTH 1.00 mm -> (none); SIZE-THICKNESS 500 µm -> (none); SIZE-WIDTH 500 µm -> (none); VOLTAGE RATING (DC) 16.0 V -> (none)
- C12: CAPACITANCE 10.0 µF -> (none); CAPACITANCE TOLERANCE ±10% -> (none); CASE/PACKAGE 0805 -> (none); DIELECTRIC CHARACTERISTIC X5R -> (none); FOOTPRINT PCB-iofq8orujrbkju2ey0y8-1 -> (none); JLCPCB Comment (none) -> 10uF 50V X5R; JLCPCB Footprint (none) -> 0805; MANUFACTURER PART NUMBER GRM21BR61H106KE43L -> (none); MPN (none) -> GRM21BR61H106KE43L; OCTOPART URL https://octopart.com/grm21br61h106ke43l-murata-52808131 -> (none); OCTOPARTID 55069f29b9a38ac1 -> (none); SIZE-LENGTH 2.00 mm -> (none); SIZE-THICKNESS 1.25 mm -> (none); SIZE-WIDTH 1.25 mm -> (none); VOLTAGE RATING (DC) 50.0 V -> (none)
- C17: CAPACITANCE 10 uF -> (none); CASE 0402 -> (none); DETAILED DESCRIPTION Multilayer Ceramic Capacitors MLCC - SMD/SMT 10UF 6.3V 20% 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 -> (none); DIELECTRIC X5R -> (none); FOOTPRINT PCB-llevxjll59guh2397ncu-2 -> (none); JLCPCB Comment (none) -> 10uF 6.3V X5R; JLCPCB Footprint (none) -> 0402; MANUFACTURER Murata -> (none); MANUFACTURER PART NUMBER GRM155R60J106ME15D -> (none); MPN (none) -> GRM155R60J106ME15D; VOLTAGE RATING DC 6.3 VDC -> (none)
- C22: JLCPCB Comment (none) -> 100nF 50V X7R; JLCPCB Footprint (none) -> 0402; MPN (none) -> GMC04X7R104K50NT
- C24: JLCPCB Comment (none) -> 10nF 35V X5R; JLCPCB Footprint (none) -> 0603; MPN (none) -> GRM188R6YA106MA73D
- C25: JLCPCB Comment (none) -> 2.2nF 10V X5R; JLCPCB Footprint (none) -> 0402; MPN (none) -> LMK105ABJ225KVHF; Part LMK105ABJ225KVHF -> (none); Requirements Low-ESR ceramic, X5R or X7R -> (none)
- C26, C28: JLCPCB Comment (none) -> 22nF 10V X5R; JLCPCB Footprint (none) -> 0805; MPN (none) -> CL21A226MPQNNNE
- C29: JLCPCB Comment (none) -> 2.2nF 10V X5R; JLCPCB Footprint (none) -> 0402; MPN (none) -> LMK105ABJ225KVHF; Part LMK105ABJ225KVHF -> (none); Requirements low-ESR ceramic chip, X7R/X5R -> (none)
- D4: JLCPCB Comment (none) -> LTST-C19HE1WT; JLCPCB Footprint (none) -> 0606; MPN (none) -> LTST-C19HE1WT; Part LTST-C19HE1WT -> (none)
- FB2: JLCPCB Comment (none) -> 30mΩ 100Ω@100MHz Ferrite Bead; JLCPCB Footprint (none) -> 0603; MPN (none) -> BLM18KG101TN1D; Part BLM18KG101TN1D -> (none)
- J1: MPN (none) -> TC2030-IDC-NL
- L2: Current Rating > 2.7A -> (none); DC resistance < 100mΩ -> (none); JLCPCB Comment (none) -> 4.7uH 3.1A 37.7mΩ; MPN (none) -> NR5040T4R7N; Part No. NR5040T4R7N -> (none)
- R13, R22, R24: CASE/PACKAGE 0402 -> (none); JLCPCB Comment (none) -> 0Ω; JLCPCB Footprint (none) -> 0402; MANUFACTURER PART NUMBER RC0402JR-100RL -> (none); MOUNTING STYLE Surface Mount -> (none); MPN (none) -> RC0402JR-100RL; OCTOPART URL https://octopart.com/rc0402jr-100rl-yageo-22251539 -> (none); OCTOPARTID 3462fc3b9917eba5 -> (none); RESISTANCE 0.0 Ω -> (none); RESISTANCE TOLERANCE ±5% -> (none)
- R19: CASE/PACKAGE 0402 -> (none); JLCPCB Comment (none) -> 120Ω 1%; JLCPCB Footprint (none) -> 0402; MANUFACTURER PART NUMBER AC0402FR-07120RL -> (none); MOUNTING STYLE Surface Mount -> (none); MPN (none) -> AC0402FR-07120RL; OCTOPART URL https://octopart.com/ac0402fr-07120rl-yageo-30510707 -> (none); OCTOPARTID 2962e1b98277f6a5 -> (none); RESISTANCE 120.0 Ω -> (none); RESISTANCE TOLERANCE ±1% -> (none)
- R2: JLCPCB Comment (none) -> 100KΩ 1%; JLCPCB Footprint (none) -> 0402; MPN (none) -> WR04X1003FTL
- RN1, RN3: JLCPCB Comment (none) -> 100KΩ; JLCPCB Footprint (none) -> 0402x2; MPN (none) -> EXB-24V104JX; Part EXB-24V104JX -> (none)
- RN2: JLCPCB Comment (none) -> 4.7KΩ; JLCPCB Footprint (none) -> 0402x2; MPN (none) -> EXB-24V472JX; Part EXB-24V472JX -> (none)
- U10: JLCPCB Comment (none) -> MX25V1006FZUI; MPN (none) -> MX25V1006FZUI
- U11: A_MAX 0.6 -> (none); B_MAX 0.23 -> (none); B_MIN 0.13 -> (none); B_NOM 0.18 -> (none); D2_NOM 0.94 -> (none); D_MAX 1.25 -> (none); D_MIN 1.15 -> (none); D_NOM 1.2 -> (none); E2_NOM 0.3 -> (none); ENOM 0.4 -> (none); E_MAX 1.25 -> (none); E_MIN 1.15 -> (none); E_NOM 1.2 -> (none); JLCPCB Comment (none) -> MIC5528-3.3YMX-TR; L_MAX 0.295 -> (none); L_MIN 0.195 -> (none); L_NOM 0.25 -> (none); MANUFACTURER MICROCHIP -> (none); MPN (none) -> MIC5528-3.3YMX-TR; PIN_COUNT 6.0 -> (none); SNAPEDA_PACKAGE_ID 7814 -> (none); STANDARD IPC 7351B -> (none)
- U4: JLCPCB Comment (none) -> STM32F042G6U6; MPN (none) -> STM32F042G6U6
- U6: JLCPCB Comment (none) -> KTD2026EWE; MPN (none) -> KTD2026EWE-TR; Manufacturer_Name Kinetic Technologies -> (none); Manufacturer_Part_Number KTD2026EWE-TR -> (none); Mouser Part Number 389-KTD2026EWETR -> (none); Mouser Price/Stock https://www.mouser.co.uk/ProductDetail/Kinetic-Technologies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 -> (none)
- U7: JLCPCB Comment (none) -> ATA6561-GBQW-N; MANUFACTURER Microchip -> (none); MAXIMUM_PACKAGE_HEIGHT 1 mm -> (none); MPN (none) -> ATA6561-GBQW-N; PARTREV B -> (none); STANDARD IPC 7351B -> (none)
- U8: JLCPCB Comment (none) -> AP63205WU-7; MPN (none) -> AP63205WU-7
