File: mikona.kicad_pcb (KiCad board)
At the start: 4 copper layers, 50 x 40 mm, 66 parts, among them J1 TC2030-IDC-NL, Q1 BSC109N10NS3G, Q2 STN3N40K3, Q3 IGB50N65S, Q4 IGB50N65S, Q5 BSS138, U1 LT3750EMSTR, U2 ZXGD3009E6, U3 NCS325, U4 PIC16F15224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

Commit message: Fix issues found during testing.
Parts:
- removed C23: 100nF, Capacitor_SMD:C_0402_1005Metric
- removed R12: 100K, Resistor_SMD:R_0402_1005Metric
- removed U2: ZXGD3009E6, Package_TO_SOT_SMD:SOT-23-6
- added C301: 10µF, Capacitor_SMD:C_0805_2012Metric, B.Cu at (133.8, 103.9)
- added C302: 100nF, Capacitor_SMD:C_0402_1005Metric, B.Cu at (131.9, 103.8)
- added RV301: 50K, Potentiometer_SMD:Potentiometer_Bourns_TC33X_Vertical, F.Cu at (137.8, 119.9)
- added U301: IX4427MTR, Package_DFN_QFN:DFN-8-1EP_3x3mm_P0.65mm_EP1.7x2.05mm, B.Cu at (129.5, 103.7)
- R3: value 40.2K -> 10K
- moved R3 2.73 mm to (134.2, 120.2), turned to 180 degrees
- moved R1 0.50 mm to (133.1, 118.1)
- turned R18 to 180 degrees
Connections:
- R3 pad 1: /Power/NMOS_DRAIN -> Net-(R3-Pad1)
Routing:
- net Net-(U1-RVOUT): track 3.24 -> 9.86 mm
- net Net-(U301-OUT_B): track 6.56 -> 1.68 mm
- net Net-(R3-Pad1): track 0.00 -> 3.30 mm
- net /Power/NMOS_DRAIN: track 2.28 -> 4.90 mm
- net +24V: track 10.1 -> 12.4 mm
- net GND: track 37.9 -> 38.4 mm, vias 38 -> 37
Other:
- outline, holes or cut-outs redrawn
- board text added: "A"
- board text added: "Ali Salehi V.2023.0.5"
- board text added: "B"
- board text added: "Cap, Mag"
- board text added: "Debug"
- board text added: "Fuse"
- board text added: "Main"
- board text added: "Vout"
- board text removed: "V.2023.0.4"

Commit message: Use parts similar to motor-driver where possible.
Parts:
- C1, C13, C301: value 10µF -> 10uF
Changed lines of the file:
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@@
     (property "JLCPCB Comment" "100nF 50V X7R")
     (property "JLCPCB Footprint" "0402")
-    (property "MPN" "GMC04X7R104K50NT")
+    (property "MPN" "GRM155R71H104KE14J")
     (property "Sheetfile" "flyback.kicad_sch")
     (property "Sheetname" "Power")
@@
     (property "JLCPCB Comment" "100pF 50V")
     (property "JLCPCB Footprint" "0402")
-    (property "MPN" "04025A101JAT2A")
+    (property "MPN" "885012205055")
     (property "Sheetfile" "flyback.kicad_sch")
     (property "Sheetname" "Power")
@@
     (property "JLCPCB Comment" "10Ω 5%")
     (property "JLCPCB Footprint" "0402")
-    (property "MPN" "ERJ-2GEJ100X")
+    (property "MPN" "ERJ-2RKF10R0X")
     (property "Sheetfile" "flyback.kicad_sch")
     (property "Sheetname" "Power")
@@
         (effects (font (size 1 1) (thickness 0.15)) (justify mirror))
     )
-    (fp_text value "10µF" (at 0 -1.68 90) (layer "B.Fab")
+    (fp_text value "10uF" (at 0 -1.68 90) (layer "B.Fab")
         (effects (font (size 1 1) (thickness 0.15)) (justify mirror))
     )
@@
     (property "JLCPCB Comment" "10Ω 5%")
     (property "JLCPCB Footprint" "0402")
-    (property "MPN" "ERJ-2GEJ100X")
+    (property "MPN" "ERJ-2RKF10R0X")
     (property "Sheetfile" "flyback.kicad_sch")
     (property "Sheetname" "Power")
@@
     (property "JLCPCB Comment" "10Ω 5%")
     (property "JLCPCB Footprint" "0402")
-    (property "MPN" "ERJ-2GEJ100X")
+    (property "MPN" "ERJ-2RKF10R0X")
     (property "Sheetfile" "flyback.kicad_sch")
     (property "Sheetname" "Power")
@@
     (property "JLCPCB Comment" "100nF 50V X7R")
     (property "JLCPCB Footprint" "0402")
-    (property "MPN" "GMC04X7R104K50NT")
+    (property "MPN" "GRM155R71H104KE14J")
     (property "Sheetfile" "flyback.kicad_sch")
     (property "Sheetname" "Power")
@@
     (property "JLCPCB Comment" "100nF 50V X7R")
     (property "JLCPCB Footprint" "0402")
-    (property "MPN" "GMC04X7R104K50NT")
+    (property "MPN" "GRM155R71H104KE14J")
     (property "Sheetfile" "logic.kicad_sch")
     (property "Sheetname" "Logic")
@@
     (property "JLCPCB Comment" "100nF 50V X7R")
     (property "JLCPCB Footprint" "0402")
-    (property "MPN" "GMC04X7R104K50NT")
+    (property "MPN" "GRM155R71H104KE14J")
     (property "Sheetfile" "flyback.kicad_sch")
     (property "Sheetname" "Power")
@@
         (effects (font (size 1 1) (thickness 0.15)) (justify mirror))
     )
-    (fp_text value "10µF" (at 0 -1.68) (layer "B.Fab")
+    (fp_text value "10uF" (at 0 -1.68) (layer "B.Fab")
         (effects (font (size 1 1) (thickness 0.15)) (justify mirror))
     )
@@
     (property "JLCPCB Comment" "100pF 50V")
     (property "JLCPCB Footprint" "0402")
-    (property "MPN" "04025A101JAT2A")
+    (property "MPN" "885012205055")
     (property "Sheetfile" "flyback.kicad_sch")
     (property "Sheetname" "Power")
@@
         (effects (font (size 1 1) (thickness 0.15)) (justify mirror))
     )
-    (fp_text value "10µF" (at 0 -1.68 90) (layer "B.Fab")
+    (fp_text value "10uF" (at 0 -1.68 90) (layer "B.Fab")
         (effects (font (size 1 1) (thickness 0.15)) (justify mirror))
     )
@@
     (property "JLCPCB Comment" "100nF 50V X7R")
     (property "JLCPCB Footprint" "0402")
-    (property "MPN" "GMC04X7R104K50NT")
+    (property "MPN" "GRM155R71H104KE14J")
     (property "Sheetfile" "logic.kicad_sch")
     (property "Sheetname" "Logic")

Commit message: Apply the MPN changes to the PCB.
Parts:
- D3: value FFSB2065BDN-F085 -> SBR40U300CTB-13
